Commit message: 241213

File: keti_workcell_description/urdf/base_ARF.urdf (robot description, URDF)
Before this commit: robot base_ARF, 16 links, 15 joints
Joints:
- removed joint ARF_jig_to_slider_base1
- removed joint ARF_slider1_s4_dummy
- removed joint base_ARF_to_ARF_jig
- removed joint world_to_base_ARF
- added joint ARF_jig_fixed: type fixed, parent base_ARF, child ARF_jig, origin xyz=-0.02392 0.03311 0.8335 rpy=0 0 -1.5709
- added joint base_ARF_fixed: type fixed, parent world, child base_ARF, origin xyz=-0.00026 0.80842 -0.0135 rpy=0 0 3.1416
- added joint s4_dummy_fixed: type fixed, parent ARF_slider1, child s4_dummy, origin xyz=-0.569 -0.06672 0.06 rpy=0 1.5709 0
- added joint slider_base1_fixed: type fixed, parent ARF_jig, child ARF_slider_base1, origin xyz=0.29294 -0.31 0.05514 rpy=-1.5709 0 0
- joint ARF_jig2_to_obj2: origin xyz=-0.01802 -0.085 0.073 rpy=0 0 -1.5709 -> xyz=-0.02828 -0.085 0.073 rpy=0 0 -1.5709
- joint ARF_jig2_to_zimmer1: axis 0 0 0 -> (none)
- joint ARF_jig2_to_zimmer2: axis 0 0 0 -> (none)
- joint ARF_slider2_jig2: axis 0 0 0 -> (none)

File: keti_workcell_description/urdf/base_DENSO.urdf (robot description, URDF)
Before this commit: robot base_DENSO, 16 links, 15 joints
Joints:
- removed joint add_axis_jig1_to_slider_base1
- removed joint add_axis_jig2_to_slider_base2
- removed joint base_DENSO_to_add_axis_jig1
- removed joint denso_jig_to_robot
- removed joint slider1_to_add_axis_jig2
- removed joint slider2_to_DENSO_jig
- removed joint world_to_base_DENSO
- added joint DENSO_jig_fixed: type fixed, parent slider2, child DENSO_jig, origin xyz=0 0.06276 0.1 rpy=-1.5709 0 0
- added joint add_axis_jig1_fixed: type fixed, parent base_DENSO, child add_axis_jig1, origin xyz=-0.02489 0.17061 0.8315 rpy=0 0 0
- added joint add_axis_jig2_fixed: type fixed, parent slider1, child add_axis_jig2, origin xyz=0 0 0.1807 rpy=-1.5709 0 0
- added joint base_DENSO_fixed: type fixed, parent world, child base_DENSO, origin xyz=-0.80034 0.81298 0 rpy=0 0 -1.5708
- added joint d_link0_fixed: type fixed, parent DENSO_jig, child d_link0, origin xyz=0 0 0 rpy=0 0 -1.5709
- added joint slider_base1_fixed: type fixed, parent add_axis_jig1, child slider_base1, origin xyz=0.37507 0 0.05482 rpy=1.5709 0 -1.5709
- added joint slider_base2_fixed: type fixed, parent add_axis_jig2, child slider_base2, origin xyz=0.35 0 0.05482 rpy=1.5709 0 -1.5709
- joint d_q3_to_end: axis 0 0 0 -> (none)
- joint denso_tool_changer_to_ATC: axis 0 0 0 -> (none)
- joint s2: origin xyz=0 0 0 rpy=0 0 0 -> xyz=-0 0 0 rpy=0 0 0

File: keti_workcell_description/urdf/base_ETC.urdf (robot description, URDF)
Before this commit: robot base_ETC, 7 links, 6 joints
Joints:
- removed joint base_ETC_to_feeder
- removed joint base_ETC_to_tool_stand
- removed joint tool_stand_to_ATC
- removed joint tool_stand_to_KRVG
- removed joint tool_stand_to_koras_2f
- removed joint world_to_base_ETC
- added joint ATC_stand_fixed: type fixed, parent tool_stand, child ATC_stand, origin xyz=-0.1258 0.1525 0.314 rpy=3.1416 0 1.5709
- added joint KRVG_stand_fixed: type fixed, parent tool_stand, child KRVG_stand, origin xyz=-0.12582 -0.1525 0.3125 rpy=3.1416 0 1.5709
- added joint base_ETC_fixed: type fixed, parent world, child base_ETC, origin xyz=-0.80481 0 -0.0135 rpy=0 0 0
- added joint feeder_fixed: type fixed, parent base_ETC, child feeder, origin xyz=-0.24992 0.19561 0.8465 rpy=0 0 0
- added joint koras_2f_stand_fixed: type fixed, parent tool_stand, child koras_2f_stand, origin xyz=-0.12582 0 0.312 rpy=3.1416 0 1.5709
- added joint tool_stand_fixed: type fixed, parent base_ETC, child tool_stand, origin xyz=0.15008 0.14561 0.8465 rpy=0 0 -1.5708

File: keti_workcell_description/urdf/base_UR.urdf (robot description, URDF)
Before this commit: robot base_UR, 12 links, 11 joints
Joints:
- removed joint UR_jig_to_UR10e
- removed joint base_UR_to_UR_jig
- removed joint link6_to_tool_changer
- removed joint tool_changer_to_koras_2f
- removed joint world_base_UR
- added joint UR_jig_fixed: type fixed, parent base_UR, child UR_jig, origin xyz=0.00017 0.04561 0.835 rpy=0 0 0
- added joint base_UR_fixed: type fixed, parent world, child base_UR, origin xyz=0 0 0.0135 rpy=0 0 0
- added joint base_link_fixed: type fixed, parent UR_jig, child base_link, origin xyz=0 0 0 rpy=0 0 3.1416
- added joint koras_2f_fixed: type fixed, parent tool_changer, child koras_2f, origin xyz=0 0 0 rpy=0 0 0
- added joint tool_fixed: type fixed, parent link6, child tool_changer, origin xyz=0 0 0.18255 rpy=0 0 0

Commit message: 241216

File: keti_workcell_description/urdf/base_ARF.urdf (robot description, URDF)
Before this commit: robot base_ARF, 16 links, 15 joints
Links:
- added link cam_jig; visual mesh filename=package://keti_workcell_description/meshes/cam_jig.STL
- added link dockingsystem; visual mesh filename=package://keti_workcell_description/meshes/docking.STL
- added link grip_adapter11; visual mesh filename=package://keti_workcell_description/meshes/grip_adapter.STL
- added link grip_adapter12; visual mesh filename=package://keti_workcell_description/meshes/grip_adapter.STL
- added link grip_adapter21; visual mesh filename=package://keti_workcell_description/meshes/grip_adapter.STL
- added link grip_adapter22; visual mesh filename=package://keti_workcell_description/meshes/grip_adapter.STL
- link base_ARF: geometry visual mesh filename=package://keti_workcell_description/meshes/base1.STL
Joints:
- added joint cam_jig_fixed: type fixed, parent dockingsystem, child cam_jig, origin xyz=-0.00103 -0.04935 0.831 rpy=0 0 -1.5709
- added joint dockingsystem_fixed: type fixed, parent base_ARF, child dockingsystem, origin xyz=-0.79918 -0.00336 -0.011 rpy=0 0 1.5709
- added joint grip_tooltip11: type fixed, parent grip_adapter11, child tooltip11, origin xyz=-0.00037 0.01437 0.019 rpy=0 0 0
- added joint grip_tooltip12: type fixed, parent grip_adapter12, child tooltip12, origin xyz=-0.00037 0.01437 0.019 rpy=0 0 0
- added joint grip_tooltip21: type fixed, parent grip_adapter21, child tooltip21, origin xyz=-0.00037 0.01437 0.019 rpy=0 0 0
- added joint grip_tooltip22: type fixed, parent grip_adapter22, child tooltip22, origin xyz=-0.00037 0.01437 0.019 rpy=0 0 0
- joint base_ARF_fixed: origin xyz=-0.00026 0.80842 -0.0135 rpy=0 0 3.1416 -> xyz=-0.00026 0.80842 0 rpy=0 0 -1.5709
- joint s5: child tooltip11 -> grip_adapter11; origin xyz=-0.00037 0.00443 -0.041 rpy=0 0 0 -> xyz=-0.00037 0.00443 -0.041 rpy=0 3.1416 0
- joint s6: child tooltip12 -> grip_adapter12; origin xyz=-0.00037 0.00443 0.041 rpy=0 3.1416 0 -> xyz=-0.00037 0.00443 0.041 rpy=0 0 0
- joint s7: child tooltip21 -> grip_adapter21
- joint s8: child tooltip22 -> grip_adapter22

File: keti_workcell_description/urdf/base_UR.urdf (robot description, URDF)
Before this commit: robot base_UR, 12 links, 11 joints
Links:
- added link HP_FeederJig; visual mesh filename=package://keti_workcell_description/meshes/HP_FeederJig.STL
Joints:
- added joint HP_FeederJig_fixed: type fixed, parent base_UR, child HP_FeederJig, origin xyz=0.52546 -0.02071 0.82 rpy=1.5709 0 -1.5709

Commit message: 241216 semi final

File: keti_workcell_description/urdf/base_ARF.urdf (robot description, URDF)
Before this commit: robot base_ARF, 22 links, 21 joints
Joints:
- joint ARF_jig_fixed: origin xyz=-0.02392 0.03311 0.8335 rpy=0 0 -1.5709 -> xyz=0.02392 0.03311 0.8335 rpy=0 0 3.14159
- joint grip_tooltip11: origin xyz=-0.00037 0.01437 0.019 rpy=0 0 0 -> xyz=-0.00037 0.01437 -0.019 rpy=0 0 0
- joint grip_tooltip12: origin xyz=-0.00037 0.01437 0.019 rpy=0 0 0 -> xyz=-0.00037 0.01437 -0.019 rpy=0 0 0
- joint grip_tooltip21: origin xyz=-0.00037 0.01437 0.019 rpy=0 0 0 -> xyz=0.00037 0.01437 -0.019 rpy=0 0 0
- joint grip_tooltip22: origin xyz=-0.00037 0.01437 0.019 rpy=0 0 0 -> xyz=0.00037 0.01437 -0.019 rpy=0 0 0
- joint s5: origin xyz=-0.00037 0.00443 -0.041 rpy=0 3.1416 0 -> xyz=0.00037 0.00443 -0.041 rpy=0 0 0
- joint s6: origin xyz=-0.00037 0.00443 0.041 rpy=0 0 0 -> xyz=0.00037 0.00443 0.041 rpy=0 3.1416 0

Commit message: 241216 vision module add

File: keti_workcell_description/urdf/base_ARF.urdf (robot description, URDF)
Before this commit: robot base_ARF, 22 links, 21 joints
Links:
- removed link cam_jig
- removed link dockingsystem
Joints:
- removed joint cam_jig_fixed
- removed joint dockingsystem_fixed
